File: schpcb/InputChannel.brd (EAGLE design)
At the start: 78 parts, among them IC1 ADA4853-3RU, IC2 4052D, IC3 4052D, IC4 OPA2354, IC7 74HC595D, K1 G6K-2F-Y, K2 G6K-2F-Y, T1 BC850, T2 BC850, T3 BC850, T4 BC850, T5 BC856ASMD, T6 BC856ASMD, T7 BC856ASMD, T8 BC856ASMD, X1 31-5431-10RFX

Commit message: Finished first outcast for inputchannel
Parts:
- C4: device passive:0603 -> passive:0402
- L1: value (none) -> 1uH
- X1: device teg4:AMP_227161 -> connectors:AMP_227161
- moved C16 76.8 mm to (53.9, 87.1)
- moved C19 72.5 mm to (50.7, 80.8)
- moved R35 64.3 mm to (35.9, 87.1)
- moved C22 48.6 mm to (25.6, 80.5), turned to 90 degrees
- moved L1 18.6 mm to (43.9, 92.6)
- moved R32 13.7 mm to (45.3, 77.4), turned to 180 degrees
- moved R25 9.50 mm to (13.3, 79.9), flipped to the bottom, turned to 90 degrees
- moved C4 9.34 mm to (41.5, 79.1), flipped to the top, turned to 270 degrees
- moved C3 8.00 mm to (42.9, 84.4), flipped to the top, turned to 0 degrees
- moved R33 7.21 mm to (46.6, 81.8), turned to 90 degrees
- moved IC4 6.78 mm to (43.0, 82.0)
- moved R24 6.56 mm to (40.7, 85.7)
- moved C18 4.86 mm to (36.3, 82.8), turned to 0 degrees
- moved R34 4.76 mm to (30.1, 79.2), turned to 270 degrees
- moved R15 4.57 mm to (27.2, 79.2), turned to 270 degrees
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Connections:
- new net OFFSETADJUST: L1.2
Routing:
- net OFFSETADJUST: track 0.00 -> 19.1 mm
- net N$27: track 0.00 -> 18.8 mm, vias 0 -> 2
- net +5V: track 98.3 -> 87.9 mm, vias 6 -> 5
- net N$10: track 72.2 -> 64.1 mm, vias 4 -> 3
- net N$24: track 8.43 -> 15.9 mm
- net -2V5A: track 51.7 -> 44.4 mm
- net N$19: track 0.00 -> 6.56 mm
- net N$31: track 0.00 -> 5.56 mm
- net +3VA: track 32.8 -> 29.2 mm
- net N$4: track 2.27 -> 5.88 mm, vias 0 -> 1
- net N$34: track 4.11 -> 7.70 mm
- net GND: track 76.2 -> 79.5 mm, vias 18 -> 23
- net N$32: track 4.06 -> 7.14 mm
- net N$21: track 4.00 -> 7.07 mm
- net N$28: track 5.85 -> 2.87 mm
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- added copper zone on layer 1, net N$22
- added copper zone on layer 3, net N$45
- added copper zone on layer 3, net N$46
- removed copper zone on layer 3, net N$50
- removed copper zone on layer 3, net N$51
- removed copper zone on layer 3, net N$52
- removed copper zone on layer 3, net N$53

Commit message: Pre release checkin
Connections:
- new net INSTOUT: IC2.14, IC2.2
Routing:
- net INSTOUT: track 0.00 -> 19.6 mm, vias 0 -> 2
Changed lines of the file:
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@@
 </polygon>
+</signal>
+<signal name="INSTOUT">
+<contactref element="IC2" pad="14"/>
+<contactref element="IC2" pad="2"/>
+<wire x1="60.1726" y1="92.6338" x2="60.1726" y2="94.107" width="0.254" layer="16"/>
+<wire x1="60.1726" y1="94.107" x2="60.833" y2="94.7674" width="0.254" layer="16"/>
+<wire x1="60.833" y1="94.7674" x2="63.7794" y2="94.7674" width="0.254" layer="16"/>
+<wire x1="63.7794" y1="94.7674" x2="64.1096" y2="94.4372" width="0.254" layer="16"/>
+<wire x1="64.1096" y1="94.4372" x2="64.1096" y2="91.6178" width="0.254" layer="16"/>
+<wire x1="64.1096" y1="91.6178" x2="64.0842" y2="91.5924" width="0.254" layer="16"/>
+<wire x1="64.0842" y1="91.5924" x2="64.0842" y2="91.567" width="0.254" layer="16"/>
+<wire x1="64.0842" y1="91.567" x2="63.373" y2="90.8558" width="0.254" layer="16"/>
+<wire x1="63.373" y1="90.8558" x2="62.8142" y2="90.8558" width="0.254" layer="16"/>
+<via x="62.8142" y="90.8558" extent="1-16" drill="0.3"/>
+<wire x1="62.8142" y1="90.8558" x2="63.0682" y2="90.678" width="0.254" layer="1"/>
+<wire x1="63.0682" y1="90.678" x2="63.246" y2="90.5002" width="0.254" layer="1"/>
+<wire x1="63.246" y1="90.5002" x2="63.246" y2="88.7222" width="0.254" layer="1"/>
+<wire x1="63.246" y1="88.7222" x2="63.373" y2="88.5952" width="0.254" layer="1"/>
+<via x="63.373" y="88.5952" extent="1-16" drill="0.3"/>
+<wire x1="63.373" y1="88.5952" x2="63.6016" y2="88.3666" width="0.254" layer="16"/>
+<wire x1="63.6016" y1="88.3666" x2="63.6016" y2="85.3186" width="0.254" layer="16"/>
+<wire x1="61.468" y1="86.4616" x2="61.4426" y2="86.487" width="0.254" layer="16"/>
+<wire x1="61.468" y1="86.4616" x2="61.468" y2="85.344" width="0.254" layer="16"/>
+<wire x1="61.468" y1="85.344" x2="61.6458" y2="85.1662" width="0.254" layer="16"/>
+<wire x1="61.6458" y1="85.1662" x2="63.4492" y2="85.1662" width="0.254" layer="16"/>
+<wire x1="63.4492" y1="85.1662" x2="63.6016" y2="85.3186" width="0.254" layer="16"/>
 </signal>
 </signals>
