File: schpcb/InputChannel.sch (EAGLE design)
At the start: 78 parts, among them IC1 ADA4853-3RU, IC2 4052D, IC3 4052D, IC4 OPA2354, IC7 74HC595D, K1 G6K-2F-Y, K2 G6K-2F-Y, T1 BC850, T2 BC850, T3 BC850, T4 BC850, T5 BC856ASMD, T6 BC856ASMD, T7 BC856ASMD, T8 BC856ASMD, X1 31-5431-10RFX

Commit message: Finished first outcast for inputchannel
Parts:
- C4: device passive:CAPC0603 -> passive:CAPC0402
- L1: value (none) -> 1uH
- X1: device teg4:1-227161-0 -> connectors:227161-8
Connections:
- new net OFFSETADJUST: L1.2
Changed lines of the file:
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@@
 <?xml version="1.0" encoding="utf-8"?>
 <!DOCTYPE eagle SYSTEM "eagle.dtd">
-<eagle version="7.2.0">
+<eagle version="7.3.0">
 <drawing>
 <settings>
@@
 <part name="P-1" library="supply1" deviceset="-12V" device="" value="-2V5A"/>
 <part name="C3" library="passive" deviceset="CAP" device="C0603" value="100nF"/>
-<part name="C4" library="passive" deviceset="CAP" device="C0603" value="100nF"/>
+<part name="C4" library="passive" deviceset="CAP" device="C0402" value="100nF"/>
 <part name="P-5" library="supply1" deviceset="-24V" device="" value="AVREFM"/>
 <part name="P-6" library="supply1" deviceset="-24V" device="" value="AVREFM"/>
@@
 <part name="C21" library="passive" deviceset="CAP" device="C0402" value="100nF"/>
 <part name="GND12" library="supply1" deviceset="GND" device=""/>
-<part name="X1" library="teg4" deviceset="?227161*" device="1-" technology="-0" value="31-5431-10RFX"/>
+<part name="X1" library="connectors" deviceset="?227161*" device="" technology="-8" value="31-5431-10RFX"/>
 <part name="GND13" library="supply1" deviceset="GND" device=""/>
 <part name="T1" library="transistor" deviceset="BC850" device=""/>
@@
 <part name="C26" library="passive" deviceset="CAP" device="C0603" value="12pF"/>
 <part name="C27" library="passive" deviceset="CAP" device="C0603" value="12pF"/>
-<part name="L1" library="rcl" deviceset="L-EU" device="L3216C"/>
+<part name="L1" library="rcl" deviceset="L-EU" device="L3216C" value="1uH"/>
 <part name="C10" library="passive" deviceset="CAP" device="C1206" value="100uF"/>
 <part name="C14" library="passive" deviceset="CAP" device="C0402" value="100nF"/>
@@
 <wire x1="91.44" y1="114.3" x2="91.44" y2="106.68" width="0.1524" layer="91"/>
 <label x="91.44" y="106.68" size="1.778" layer="95"/>
+<pinref part="L1" gate="G$1" pin="2"/>
 </segment>
 </net>
@@
 </sheet>
 </sheets>
+<errors>
+</errors>
 </schematic>
 </drawing>

Commit message: Pre release checkin
Connections:
- new net INSTOUT: IC2A.X1, IC2A.Y2
Other:
- moved on the sheet: R4
Changed lines of the file:
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@@
 <grid distance="0.1" unitdist="inch" unit="inch" style="lines" multiple="1" display="no" altdistance="0.01" altunitdist="inch" altunit="inch"/>
 <layers>
-<layer number="1" name="Top" color="4" fill="1" visible="yes" active="no"/>
-<layer number="2" name="Route2" color="1" fill="3" visible="yes" active="no"/>
-<layer number="3" name="Route3" color="4" fill="3" visible="yes" active="no"/>
-<layer number="14" name="Route14" color="1" fill="6" visible="yes" active="no"/>
-<layer number="15" name="Route15" color="4" fill="6" visible="yes" active="no"/>
-<layer number="16" name="Bottom" color="1" fill="1" visible="yes" active="no"/>
-<layer number="17" name="Pads" color="2" fill="1" visible="yes" active="no"/>
-<layer number="18" name="Vias" color="2" fill="1" visible="yes" active="no"/>
-<layer number="19" name="Unrouted" color="6" fill="1" visible="yes" active="no"/>
-<layer number="20" name="Dimension" color="15" fill="1" visible="yes" active="no"/>
-<layer number="21" name="tPlace" color="7" fill="1" visible="yes" active="no"/>
-<layer number="22" name="bPlace" color="7" fill="1" visible="yes" active="no"/>
-<layer number="23" name="tOrigins" color="15" fill="1" visible="yes" active="no"/>
-<layer number="24" name="bOrigins" color="15" fill="1" visible="yes" active="no"/>
-<layer number="25" name="tNames" color="7" fill="1" visible="yes" active="no"/>
-<layer number="26" name="bNames" color="7" fill="1" visible="yes" active="no"/>
-<layer number="27" name="tValues" color="7" fill="1" visible="yes" active="no"/>
-<layer number="28" name="bValues" color="7" fill="1" visible="yes" active="no"/>
+<layer number="1" name="Top" color="4" fill="1" visible="no" active="no"/>
+<layer number="2" name="Route2" color="1" fill="3" visible="no" active="no"/>
+<layer number="3" name="Route3" color="4" fill="3" visible="no" active="no"/>
+<layer number="14" name="Route14" color="1" fill="6" visible="no" active="no"/>
+<layer number="15" name="Route15" color="4" fill="6" visible="no" active="no"/>
+<layer number="16" name="Bottom" color="1" fill="1" visible="no" active="no"/>
+<layer number="17" name="Pads" color="2" fill="1" visible="no" active="no"/>
+<layer number="18" name="Vias" color="2" fill="1" visible="no" active="no"/>
+<layer number="19" name="Unrouted" color="6" fill="1" visible="no" active="no"/>
+<layer number="20" name="Dimension" color="15" fill="1" visible="no" active="no"/>
+<layer number="21" name="tPlace" color="7" fill="1" visible="no" active="no"/>
+<layer number="22" name="bPlace" color="7" fill="1" visible="no" active="no"/>
+<layer number="23" name="tOrigins" color="15" fill="1" visible="no" active="no"/>
+<layer number="24" name="bOrigins" color="15" fill="1" visible="no" active="no"/>
+<layer number="25" name="tNames" color="7" fill="1" visible="no" active="no"/>
+<layer number="26" name="bNames" color="7" fill="1" visible="no" active="no"/>
+<layer number="27" name="tValues" color="7" fill="1" visible="no" active="no"/>
+<layer number="28" name="bValues" color="7" fill="1" visible="no" active="no"/>
 <layer number="29" name="tStop" color="7" fill="3" visible="no" active="no"/>
 <layer number="30" name="bStop" color="7" fill="6" visible="no" active="no"/>
@@
 <layer number="35" name="tGlue" color="7" fill="4" visible="no" active="no"/>
 <layer number="36" name="bGlue" color="7" fill="5" visible="no" active="no"/>
-<layer number="37" name="tTest" color="7" fill="1" visible="yes" active="no"/>
-<layer number="38" name="bTest" color="7" fill="1" visible="yes" active="no"/>
+<layer number="37" name="tTest" color="7" fill="1" visible="no" active="no"/>
+<layer number="38" name="bTest" color="7" fill="1" visible="no" active="no"/>
 <layer number="39" name="tKeepout" color="4" fill="11" visible="no" active="no"/>
 <layer number="40" name="bKeepout" color="1" fill="11" visible="no" active="no"/>
@@
 <layer number="44" name="Drills" color="7" fill="1" visible="no" active="no"/>
 <layer number="45" name="Holes" color="7" fill="1" visible="no" active="no"/>
-<layer number="46" name="Milling" color="3" fill="1" visible="yes" active="no"/>
-<layer number="47" name="Measures" color="7" fill="1" visible="yes" active="no"/>
-<layer number="48" name="Document" color="7" fill="1" visible="yes" active="no"/>
-<layer number="49" name="Reference" color="7" fill="1" visible="yes" active="no"/>
-<layer number="50" name="dxf" color="7" fill="1" visible="yes" active="no"/>
-<layer number="51" name="tDocu" color="7" fill="1" visible="yes" active="no"/>
-<layer number="52" name="bDocu" color="7" fill="1" visible="yes" active="no"/>
+<layer number="46" name="Milling" color="3" fill="1" visible="no" active="no"/>
+<layer number="47" name="Measures" color="7" fill="1" visible="no" active="no"/>
+<layer number="48" name="Document" color="7" fill="1" visible="no" active="no"/>
+<layer number="49" name="Reference" color="7" fill="1" visible="no" active="no"/>
+<layer number="50" name="dxf" color="7" fill="1" visible="no" active="no"/>
+<layer number="51" name="tDocu" color="7" fill="1" visible="no" active="no"/>
+<layer number="52" name="bDocu" color="7" fill="1" visible="no" active="no"/>
 <layer number="90" name="Modules" color="5" fill="1" visible="yes" active="yes"/>
 <layer number="91" name="Nets" color="2" fill="1" visible="yes" active="yes"/>
@@
 </plain>
 <instances>
-<instance part="IC1" gate="A" x="139.7" y="175.26"/>
+<instance part="IC1" gate="A" x="139.7" y="175.26" smashed="yes">
+<attribute name="NAME" x="144.78" y="177.8" size="1.778" layer="95"/>
+<attribute name="VALUE" x="139.7" y="181.61" size="1.778" layer="96"/>
+</instance>
 <instance part="IC1" gate="B" x="218.44" y="175.26"/>
 <instance part="IC1" gate="C" x="261.62" y="175.26"/>
@@
 <instance part="R2" gate="G$1" x="134.62" y="154.94" rot="R90"/>
 <instance part="R3" gate="G$1" x="134.62" y="142.24" rot="R90"/>
-<instance part="R4" gate="G$1" x="167.64" y="175.26" rot="R180"/>
+<instance part="R4" gate="G$1" x="160.02" y="175.26" smashed="yes" rot="R180">
+<attribute name="NAME" x="164.592" y="178.816" size="1.778" layer="95" rot="R180"/>
+<attribute name="VALUE" x="164.338" y="176.022" size="1.4224" layer="96" rot="R180"/>
+</instance>
 <instance part="R5" gate="G$1" x="220.98" y="162.56"/>
 <instance part="R6" gate="G$1" x="213.36" y="154.94" rot="R90"/>
@@
 <segment>
 <pinref part="R1" gate="G$1" pin="P$2"/>
-<wire x1="147.32" y1="162.56" x2="162.56" y2="162.56" width="0.1524" layer="91"/>
-<wire x1="162.56" y1="162.56" x2="162.56" y2="175.26" width="0.1524" layer="91"/>
+<wire x1="147.32" y1="162.56" x2="154.94" y2="162.56" width="0.1524" layer="91"/>
+<wire x1="154.94" y1="162.56" x2="154.94" y2="175.26" width="0.1524" layer="91"/>
 <pinref part="IC1" gate="A" pin="OUT"/>
 <pinref part="R4" gate="G$1" pin="P$2"/>
-<junction x="162.56" y="175.26"/>
-<wire x1="162.56" y1="175.26" x2="147.32" y2="175.26" width="0.1524" layer="91"/>
+<junction x="154.94" y="175.26"/>
+<wire x1="154.94" y1="175.26" x2="147.32" y2="175.26" width="0.1524" layer="91"/>
 </segment>
 </net>
@@
 <segment>
 <pinref part="R4" gate="G$1" pin="P$1"/>
+<wire x1="167.64" y1="175.26" x2="175.26" y2="175.26" width="0.1524" layer="91"/>
 <wire x1="175.26" y1="175.26" x2="175.26" y2="177.8" width="0.1524" layer="91"/>
 <wire x1="175.26" y1="177.8" x2="180.34" y2="177.8" width="0.1524" layer="91"/>
@@
 </segment>
 </net>
+<net name="INSTOUT" class="0">
+<segment>
+<pinref part="IC2" gate="A" pin="X1"/>
+<wire x1="180.34" y1="187.96" x2="172.72" y2="187.96" width="0.1524" layer="91"/>
+<label x="162.56" y="187.96" size="1.778" layer="95"/>
+</segment>
+<segment>
+<pinref part="IC2" gate="A" pin="Y2"/>
+<wire x1="180.34" y1="172.72" x2="177.8" y2="172.72" width="0.1524" layer="91"/>
+<label x="167.64" y="172.72" size="1.778" layer="95"/>
+</segment>
+</net>
