File: schpcb/LabFriendMain1.brd (EAGLE design)
At the start: 100 x 100.1 mm, 299 parts, among them IC1 TPS62560, IC10 TPS62560, IC11 TPS62560, IC12 TPS62560, IC14 TPS72301, IC18 LM358D, IC19 LM358D, IC2 25px80, IC20 PCM3010, IC21 TS922, IC23 TS922, IC24 4052D, IC25 ADS1112, IC26 MT41J128M8, IC3 SI8462, IC4 FT232H, IC5 ADC08200, IC6 ADC08200, IC8 93LC56SM, IC9 74LVC8T245, Q1 12MHz, U2 6SLX9FTG256, X1 MINI-USB-32005-201

Commit message: current state
Parts:
- added C100, C102: 2n2, passive:0603
- added C101, C114, C98, C99: 330pF, passive:0603
- added C103, C113: 47uF, passive:1206
- added C115, C116, C145, C146, C147, C193, C197, C198, C96, C97: 100nF, passive:0402
- added C148, C150: (no value), passive:0402
- added C149: 100pF, teg2:0603
- added C151, C152: 47pF, teg2:0603
- added C153, C154: 100n, teg2:0603
- added C155, C156, C160: 100nF, teg2:0603
- added C157, C158, C159, C161: 100µF, rcl:CT6032
- added C162, C173, C178, C181, C188, C189, C191, C196, C199: 1uF, passive:0603
- added C163, C174: 22pF, passive:0603
- added C164: 100uF, passive:0402
- added C165, C171, C177, C179, C180, C182, C183, C184, C185, C186, C187, C192, C194, C200: 10uF, passive:0603
- added C166: 470nF, passive:1206
- added C167: 470nF, passive:0402
- added C168, C169, C170, C175, C176: 10µF, passive:0603
- added C172, C190, C195: 10nF, passive:0603
- added D1, D2, D3, D4, D5, D6: SK14, diode:DO214AC
- added IC13: AK4621, data-converters:VSOP30
- added IC15: LME49721, linear:SO08
- added IC16: NE5532, linear:SO08
- added IC17: OPA2134, linear:SO08
- added IC22: 4052D, 40xx:SO16
- added IC27: 74HCT132D, 74xx-eu:SO14
- added IC28: TPS72301, seabed:SOT23-5L
- added IC29: (no value), seabed:SOT23-6L
- added IC30: LM8272, linear:MSOP08
- added IC31: LMV358MM, linear:MSOP08
- added L11, R153, R163, R164, R166, R167, R175, R176: (no value), passive:0603
- added Q2, Q3: FDN335N, transistor-small-signal:SOT23
- added R132, R133, R134: 1k5, passive:0603
- added R135, R136, R137, R138: 3k, passive:0603
- added R139, R140, R141, R142: 22R, teg2:0603
- added R143, R144: 10k, passive:0603
- added R145, R147, R148, R149, R181, R182, R189, R190, R191, R194, R196, R200, R58, R74: 4k7, passive:0603
- added R146, R150: 220k, passive:0603
- added R151: 4k7, teg2:0603
- added R152: 100R, teg2:0603
- added R154: 1M, passive:0603
- added R155, R187, R188: 100k, passive:0603
- added R156: 1k, passive:0603
- added R157, R158: 10k, teg2:0603
- added R159, R160: 1.54k, teg2:0603
- added R161, R162: 150, teg2:0603
- added R165, R168, R172, R173, R174, R177, R178, R179, R180, R183, R184, R185, R186, R192, R193: 0R1, passive:0603
- added R169: 1M, passive:0402
- added R170, R171: 820k, passive:0603
- added R195: 1k3, passive:0603
- added R197: 5k1, passive:0603
- added R198: 68k, passive:0603
- added R199: 15k, passive:0603
- added R56, R57: 200, passive:0603
- added T1: EFD15DCDCPM5P33EFD15, transformers:B66414-W1008-D1
- C1, C2, C3, C78, C79, C80, C82, C88, C92, C93, R107, R112, R14, R15, R16, R17, R18, R19, R20, R21, R38, R39, R40, R41, R42, R43, R44, R45, R46, R47, R52, R53, R65, R66, R75, R76, R77, R78, R93: device teg2:0603 -> passive:0603
- C104, C105, C112, R10, R100, R101, R102, R103, R11, R12, R22, R23, R24, R25, R26, R27, R28, R29, R30, R31, R32, R33, R34, R35, R36, R37, R4, R5, R6, R79, R8, R88, R89, R9, R97, R98, R99: device teg2:0603 -> passive:0402
- C106, C107, C108, C109, C110, C111, C118, C125, C13, C134, C137, C138, C14, C140, C141, C28, C32, C33, C58, C60, C61, C62, C63, C64, C65, C67, C68, C69, C76, C77: device rcl:C0402 -> passive:0402
- C11: device rcl:C1206 -> passive:1206
- C117, C126: value 10uF -> 100nF; device rcl:C0603K -> passive:0402
- C119, C29, C30, C31, C36, C37, C39, C40, C41, C42, C43, C44, C45, C46, C47, C48, C49, C50, C52, C53, C54, C55, C56, C74: device rcl:C0603K -> passive:0603
- C12, C57, C59, C66, C70: device rcl:C0603 -> passive:0603
- C120, C73: value 100nF -> 10uF; device rcl:C0402 -> passive:0603
- C121, C123: value 10uF -> 330pF; device rcl:C0603K -> passive:0603
- C122, C124: value 100nF -> 330pF; device rcl:C0402 -> passive:0603
- C127: value 10uF -> 10nF; device rcl:C0603K -> passive:0603
- C128: value 200pF -> 330pF; device rcl:C0603K -> passive:0603
- C129, C130, C131, C132, C133: value 200pF -> 47uF; device rcl:C0603K -> passive:1206
- C135, C136: value 10uF -> 47uF; device rcl:C0603K -> passive:1206
- C21, C23, C35: value 4u7 -> 100uF; device rcl:C0603K -> passive:1206
- C22, C25: value 4u7 -> 470nF; device rcl:C0603K -> passive:0402
- C24: value 4u7 -> 10uF; device rcl:C0603K -> passive:0603
- C26, C38: device rcl:C0603K -> passive:0402
- C34: value 470nF -> 10uF; device rcl:C0402 -> passive:0603
- C71: value 10uF -> 100uF; device rcl:C0603 -> passive:1206
- C72: value 100nF -> 470nF; device rcl:C0402 -> passive:0402
- C81: value 33pF -> 10uF; device teg2:0603 -> passive:0603
- C83, C87: value 10µF -> 10nF; device teg2:0603 -> passive:0603
- C84: value 33pF -> 1uF; device teg2:0603 -> passive:0603
- C85: value 10µF -> 22pF; device teg2:0603 -> passive:0603
- C86: value 10µF -> 10uF; device teg2:0603 -> passive:0603
- C91, C95: device passive:0402 -> passive:0603
- IC11, IC12: value TPS62560 -> (none); device seabed:SOT23-5L -> seabed:SOT23-6L
- IC18: value LM358D -> LM8272; device linear:SO08 -> linear:MSOP08
- IC19: value LM358D -> LMV358MM; device linear:SO08 -> linear:MSOP08
- IC20: value PCM3010 -> ISL54405IRTZ; device parts2004:SSOP24 -> switch_mux:TQFN3X3
- IC21: value TS922 -> NE5532
- IC23: value TS922 -> LME49721
- IC24: value 4052D -> 74HC00D; device 40xx:SO16 -> 74xx-eu:SO14
- L10, L8, L9: value 4.7uH -> (none); device rcl:L3216C -> passive:0603
- R105, R94: value 47R -> 200; device teg2:0603 -> passive:0603
- R106: value 47R -> 1k5; device teg2:0603 -> passive:0603
- R48, R50: value 820k -> 0R1; device teg2:0603 -> passive:0603
- R49, R51: value 180k -> 0R1; device teg2:0603 -> passive:0603
- R54, R55: value RESR0603 -> (none)
- R61, R63: value 51k -> 68k; device teg2:0603 -> passive:0603
- R62, R64: value 22k -> 15k; device teg2:0603 -> passive:0603
- R83, R91: value 10M -> 4k7; device teg2:0603 -> passive:0603
- R84, R85: value 6k8 -> 4k7; device teg2:0603 -> passive:0603
- R86, R87: value 47R -> 600R
- R92: value 47R -> 4k7; device teg2:0603 -> passive:0603
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Connections:
- removed net +5V/1: C3.2, C80.2, C83.2, C86.2, IC1.1, IC1.3, IC10.1, IC10.3, IC11.1, IC11.3, IC12.1, IC12.3
- removed net -2V2: C105.2, C137.1, C141.2, IC18.4, IC23.4, IC24.7
- removed net ASEL1: IC24.9
- removed net HPADSPICS: IC3.11, U2.P7
- new net +3.6VBR: C162.2, C3.2, C80.2, C84.2, IC1.1, IC1.3, IC10.1, IC10.3, IC11.1, IC11.3, IC12.1, IC12.3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
- new net +3.6VI: C94.2, IC7.1, IC7.3, R179.1
- new net +5.5V: C156.1, C157.+, D1.C, D2.C, R178.1
- new net +5.5VI: C173.2, IC29.1, IC29.3, R178.2
- new net -2.5VI: C93.1, IC14.5, R174.1, R52.2
- new net -2V5: C176.1, C198.2, R174.2
- new net -5.5V: C155.2, C158.-, D3.A, D4.A, R172.1
- new net 1V2REFAD0: C111.1, IC5.10, L10.2
- new net 1V2REFAD1: C108.1, IC6.10, L9.2
- new net 2V8REFAD0: C109.1, IC5.3, L11.2
- new net 2V8REFAD1: C106.1, IC6.3, L8.2
- new net AUADCINL: C132.1, IC17.6, IC17.7, R149.2
- new net AUADCINR: C130.1, IC17.1, IC17.2, R147.2
- new net AUBIAS: C133.2, C134.2, IC15.2, IC15.5, IC23.3, IC23.5, R143.1, R144.2
- new net AUPDN: IC13.21
- new net AU_CCLK: IC13.18
- new net AU_CDTI: IC13.17
- new net AU_CSN: IC13.19
- new net AU_OVFL: IC13.16
- new net AU_OVFR: IC13.15
- new net AVREFM: C192.1, R192.2
- new net CMPMEAS_+: IC20.11, R153.1, R154.1, R155.1, R156.1, SV4.1
- new net CMPMEAS_-: IC20.9, IC22.3
- new net CMPMEAS_A: IC22.10
- new net CMPMEAS_B: IC22.9
- new net CMPMEAS_EN: IC22.6
- new net CMPMEAS_O: IC22.13, R152.2
- new net EXVOI: IC19.7, R185.1, R75.1
- new net LAD13OO: U2.P11
- new net LADVREF: C167.1, R169.2, U2.M10, U2.T5
- new net LAVIOI: C188.2, IC19.1, R186.1, R66.1
- new net N$111: C101.1, IC21.2, R94.2
- new net N$125: C121.1, IC23.6, R106.1, R135.2
- new net N$152: C122.1, IC15.3, R134.1, R137.2
- new net N$154: C123.1, IC15.6, R133.1, R136.2
- new net N$156: C124.1, IC23.2, R132.1, R138.2
- new net N$158: C127.2, IC13.4, R140.1
- new net N$160: C127.1, IC13.5, R139.2
- new net N$161: C128.1, IC13.3, R142.2
- new net N$166: C128.2, IC13.2, R141.1
- new net N$167: C129.2, R135.1
- new net N$168: C130.2, R138.1
- new net N$169: C131.2, R136.1
- new net N$170: C132.2, R137.1
- new net N$171: C131.1, IC16.7, R148.1
- new net N$172: IC17.5, IC20.3, R150.2
- new net N$173: IC17.3, IC20.2, R146.2
- new net N$174: C146.2, IC20.13
- new net N$175: C129.1, IC16.1, R145.1
- new net N$176: IC16.2, R145.2, R147.1
- new net N$177: IC16.6, R148.2, R149.1
- new net N$178: IC20.10, R151.1
- new net N$179: IC22.1, IC22.12, R153.2
- new net N$180: IC22.14, IC22.5, R154.2
- new net N$181: IC22.15, IC22.2, R155.2
- new net N$182: IC22.11, IC22.4, R156.2
- new net N$183: C148.2, C150.1, IC22.8
- new net N$184: IC27.1, IC27.2, R157.1
- new net N$185: IC24.4, IC24.5, IC27.3
- new net N$186: C149.1, R157.2, R158.1
- new net N$187: C149.2, IC24.1, IC24.2, IC24.6
- new net N$188: IC24.3, IC27.12, IC27.4, IC27.5, R158.2, R160.1
- new net N$189: C151.2, IC27.13, R160.2
- new net N$190: IC27.6, IC27.9, R159.1
- new net N$191: C152.2, IC27.10, R159.2
- new net N$192: IC24.10, IC24.9, IC27.8
- new net N$193: IC24.12, IC24.13, IC27.11
- new net N$194: IC24.11, R161.1
- new net N$195: IC24.8, R162.1
- new net N$196: Q3.1, R162.2
- new net N$197: D2.A, D3.C, T1.8
- new net N$198: D1.A, D4.C, T1.7
- new net N$199: Q2.3, T1.1
- new net N$200: Q2.1, R161.2
- new net N$201: Q3.3, T1.3
- new net N$202: D5.A, T1.5
- new net N$203: D6.A, T1.6
- new net N$204: R195.2, R197.1
- new net N$205: R43.1, U2.B8
- new net N$206: C81.2, C85.2, IC11.6, R163.2, R165.1
- new net N$207: C85.1, IC11.5, R163.1, R164.2
- new net N$208: C163.2, C86.2, IC12.6, R166.2, R168.1
- new net N$209: C163.1, IC12.5, R166.1, R167.2
- new net N$210: R169.1, U2.N6
- new net N$211: C169.1, IC28.5, R170.2, R173.1
- new net N$212: IC28.4, R170.1, R171.2
- new net N$213: C190.1, IC30.1, R189.1, R192.1
- new net N$214: C172.2, IC29.4
- new net N$215: C171.2, C174.2, IC29.6, R175.2, R177.1
- new net N$216: C174.1, IC29.5, R175.1, R176.2
- new net N$217: C190.2, IC30.2, R189.2
- new net N$218: C195.1, IC30.7, R191.2, R193.1, R194.1
- new net N$219: C195.2, IC30.6, R194.2
- new net N$220: C196.1, IC30.5, R196.1, R197.2
- new net N$221: C199.1, IC31.6, R198.2, R199.1
- new net N$223: C200.1, R199.2, R200.1
- new net N$23: C191.1, IC30.3, R190.2, R191.1
- new net N$83: C135.2, R58.1
- new net N$88: C136.2, R74.1
- new net OFFSETCH0I: C178.1, IC18.1, R183.1, R61.1
- new net OFFSETCH1I: C181.2, IC18.7, R184.1, R63.1
- new net PWMEXVO: R188.2
- new net PWMLA: R200.2
- new net PWMLAVIO: R187.2
- new net PWMOFFS0: R181.2
- new net PWMOFFS1: R182.2
- new net V-: IC31.4
- net +3.6V: now also C160.1, C161.+, D5.C, D6.C, IC31.8, R179.2, R48.1; no longer C94.2, IC7.1, IC7.3
- net +3V3: now also C116.1, C117.1, C147.2, C164.2, C165.2, C166.2, IC13.24, IC13.25, IC20.14, R165.2, U2.A4, U2.B13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; no longer C125.1, C21.1, C81.2, IC20.15, IC20.17, IC20.19, IC20.7, IC20.8, L8.2, R48.2
- net +5V: now also C104.2, C115.2, C119.2, C125.1, C126.1, C138.1, C141.1, C145.1, C148.1, C170.2, C96.1, IC13.6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; no longer C123.1, C124.1, C134.1, C140.1, IC20.21, IC20.5, IC24.16
- net +UB: now also C153.2, C154.2, C159.+, IC24.14, IC27.14, R51.2, T1.2; no longer C74.1, L6.1
- net -5V: now also C105.2, C137.1, C140.1, C150.2, C175.1, C97.1, IC16.4, IC17.4, IC18.4, IC21.4, IC22.7, R173.2; no longer C93.1, IC14.5, R52.2
- net 1V2REF: now also C194.1, IC31.5, L10.1, L9.1, R193.2; no longer C108.1, C111.1, IC24.15, IC24.2, IC5.10, IC6.10
- net 2V8REF: now also C177.2, C193.2, IC30.8, L11.1, L8.1, R180.1, R190.1, R195.1; no longer C106.1, C109.1, IC5.3, IC6.3
- net 3V3A: now also C197.2, R168.2; no longer C104.2, C138.2, C87.2, IC18.8, IC23.8, L10.2
- net ADA0: now also U2.E16; no longer U2.F14
- net ADA1: now also U2.E15; no longer U2.F13
- net ADA4: now also U2.C16; no longer U2.G11
- net ADA5: now also U2.C15; no longer U2.F12
- net ADAC: now also U2.F15; no longer U2.C16
- net ADAP: now also U2.F16; no longer U2.C15
- net ADB0: now also U2.K14; no longer U2.G12
- net ADB1: now also U2.K16; no longer U2.H16
- net ADB2: now also U2.K15; no longer U2.H15
- net ADB3: now also U2.J16; no longer U2.G16
- net ADB4: now also U2.H16; no longer U2.G14
- net ADB5: now also U2.H15; no longer U2.F16
- net ADB6: now also U2.G16; no longer U2.F15
- net ADB7: now also U2.F14; no longer U2.E16
- net ADBC: now also U2.L16; no longer U2.E15
- net AINL: no longer R92.2
- net AINR: now also R151.2; no longer R106.2, R93.2
- net ASEL0: no longer IC24.10
- net EXVO: now also C184.1, R185.2; no longer IC19.7, R75.1
- net GND: now also C114.1, C115.1, C116.2, C118.1, C119.1, C120.1, C126.2, C133.1, C134.1, C138.2, C141.2, C145.2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; no longer C118.2, C119.2, C120.2, C121.2, C122.2, C123.2, C124.2, C128.2, C129.2, C130.2, C131.2, C132.2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
- net GNDIO: now also C151.1, C152.1, C153.1, C154.1, C159.-, IC24.7, IC27.7, Q2.2, Q3.2
- net I2SBCK: now also IC13.12; no longer IC20.11, U2.M6
- net I2SDATAIN: now also IC13.14; no longer IC20.12
- net I2SLRCK: now also IC13.11; no longer IC20.10, U2.N6
- net I2SSCLK: now also IC13.10; no longer IC20.16
- net LAD0: now also U2.T9
- net LAD1: now also U2.P7
- net LAD10: now also U2.P6; no longer U2.H13
- net LAD11: now also U2.N8; no longer U2.H11
- net LAD13: now also U2.P9; no longer U2.P11
- net LAD2: now also U2.T8
- net LAD3: now also U2.T7
- net LAD4: now also U2.R7
- net LAD5: now also U2.T6; no longer U2.K14
- net LAD6: now also U2.R5; no longer U2.J13
- net LAD7: now also U2.T4; no longer U2.J12
- net LAD8: now also U2.N5; no longer U2.J11
- net LAD9: now also U2.P5; no longer U2.H14
- net LAVIO: now also C185.1, R186.2; no longer IC19.1, R66.1
- net LOGICOFFSET: now also C199.2, IC31.7, R198.1
- net MSTCLK: now also U2.B10; no longer U2.T8
- net N$100: now also C187.1, R188.1
- net N$107: now also C189.1
- net N$109: now also C101.2, IC21.1, R152.1, R85.2, R86.1; no longer IC20.23, R84.1
- net N$11: now also C83.2, IC11.4; no longer R41.1, U2.N5
- net N$113: now also C114.2, IC21.3, R105.2; no longer C135.1, IC21.1, IC21.2
- net N$114: now also C102.2, R85.1, R91.2, R94.1; no longer C126.1, IC20.2
- net N$115: now also C121.2, IC23.7, R106.2, R141.2; no longer C127.1, IC20.1
- net N$116: now also C102.1, R105.1, R92.2, R93.2; no longer C131.1, C132.1, C133.1, IC21.3, R84.2
- net N$118: now also C103.2, R91.1; no longer C136.1, IC21.6, IC21.7
- net N$119: now also C113.2, R92.1; no longer C135.2, R86.1
- net N$12: now also R41.1, U2.C9; no longer R42.1, U2.T5
- net N$120: now also C103.1, IC13.29; no longer C136.2, R87.1
- net N$121: now also IC13.13; no longer IC20.13
- net N$122: now also C113.1, IC13.30; no longer C127.2, IC23.1, IC23.2
- net N$123: now also C136.1, IC13.28; no longer IC23.3, IC24.13, R91.2
- net N$124: now also C135.1, IC13.27; no longer C126.2, IC23.6, IC23.7
- net N$13: now also R42.1, U2.A9; no longer R43.1, U2.M7
- net N$14: now also C98.1, IC21.6, R56.2; no longer IC20.22, R85.1
- net N$141: now also C124.2, IC23.1, R132.2, R142.1; no longer IC23.5, IC24.3, R83.2
- net N$143: now also C123.2, IC15.7, R133.2, R140.2; no longer IC24.14, R92.1, R94.2
- net N$145: now also C118.2, C120.2, IC13.1; no longer IC24.5, R105.2, R106.1
- net N$146: now also C122.2, IC15.1, R134.2, R139.1; no longer IC24.1, R93.1
- net N$147: now also IC20.12; no longer IC24.12
- net N$15: now also U2.A7; no longer U2.R5
- net N$6: now also U2.A10; no longer U2.P5
- net N$76: now also C99.2, IC21.5, R57.2; no longer C117.1, C120.1, IC20.24
- net N$77: now also C98.2, IC21.7, R83.2, R87.1; no longer C118.1, C119.1, IC20.4
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Routing:
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- added copper zone on layer 3, net +3V3
- added copper zone on layer 2, net GND
- added copper zone on layer 3, net VCCDDR3
- added copper zone on layer 3, net VCCINT
- removed copper zone on layer 2, net +3V3
- removed copper zone on layer 2, net 3V3A
- removed copper zone on layer 1, net GND
- removed copper zone on layer 3, net GND
- removed copper zone on layer 1, net GNDIO
- removed copper zone on layer 3, net N$262
- removed copper zone on layer 2, net VCCDDR3
- removed copper zone on layer 1, net VCCIO
Other:
- board size 100 x 100.1 mm -> 128 x 411.1 mm

Commit message: Pre release checkin
Parts:
- added C201, C202, C203: 10nF, passive:0402
- added C204, C206, C207, C208, C209, C210, C218, C219, C220, C221, C225, C226, C227, C231, C232, C233, C234, C235, C243, C244, C245, C246, C250, C251, C252, C255, C256: 100nF, passive:0402
- added C205, C230: 10uF, passive:0603
- added C211, C236: 100nF, passive:0603
- added C212, C214, C217, C222, C223, C237, C239, C242, C247, C248: 12pF, passive:0603
- added C213, C216, C238, C241: 6/30, rcl:CTRIMTZBX4
- added C215, C240: 220pF, passive:0603
- added C224, C249: 100uF, passive:1206
- added C228, C229, C253, C254: 1pF, passive:0603
- added IC32: ADS1118IDGSR, data-converters:MSOP10
- added IC33, IC38: ADA4853-3RU, teg4:SO14
- added IC34, IC35, IC39, IC40: 4052D, 40xx:SO16
- added IC36, IC41: OPA2354, linear:MSOP08
- added IC37, IC42, IC44: 74HC595D, 74xx-eu:SO16
- added IC43: LM321MF, linear:SOT23-5
- added K1, K2, K3, K4: G6K-2F-Y, relay:G6K-2F-Y
- added L12, L14: 1uH, rcl:L3216C
- added R201: NC, passive:0402
- added R202: 91k, passive:0603
- added R203, R218, R219, R220, R254, R255, R256: 10k, passive:0603
- added R204, R205: 27k, passive:0603
- added R206, R207: 22k, passive:0603
- added R208, R244: 200R, passive:0603
- added R209, R245: 30R, passive:0603
- added R210, R246: 20R, passive:0603
- added R211, R214, R217, R237, R239, R247, R250, R253, R273, R275, R278, R279: 22R, passive:0603
- added R212, R215, R216, R229, R230, R238, R248, R251, R252, R265, R266, R274, R300: 300R, passive:0603
- added R213, R249, R277: 100R, passive:0603
- added R221, R222, R257, R258: 30k, passive:0603
- added R223, R224, R259, R260: 470k, passive:0603
- added R225, R261: 51k, passive:0603
- added R226, R262: 39k, passive:0603
- added R227, R263: 910k, passive:0603
- added R228, R264: 1k, passive:0603
- added R231, R267: 7R5, passive:0603
- added R232, R233, R234, R235, R236, R268, R269, R270, R271, R272: 10R, passive:0603
- added R240, R276: 1R, passive:0603
- added R241: 100R, passive:0402
- added R242, R243: 47R, passive:0603
- added R280: 1k, passive:0402
- added R281: 2k2, passive:0402
- added R282: 50R, passive:0603
- added R283, R285, R292, R293, R294, R295, R296, R297, R298: 1k6, passive:0603
- added R284, R286, R287, R288, R289, R290, R291: 820R, passive:0603
- added R299: 39R, passive:0603
- added SV5: 3x1 Pinheader, con-lstb:MA03-1
- added T10, T11, T14, T16, T2, T3, T4, T8: BC850, transistor:SOT23
- added T12, T13, T15, T17, T5, T6, T7, T9: BC856ASMD, transistor-pnp:SOT23-BEC
- added X2, X3: 31-5431-10RFX, connectors:AMP_227161
- C10, C139, C142, C143, C144, C15, C16, C17, C18, C20, C8, C9: device rcl:C0402 -> passive:0402
- C12, C43, C44, C46, C48, C74: value 4.7uF -> 10uF
- C128: value 330pF -> 10nF
- C148, C150: value (none) -> 100nF
- C149, C151, C152, R104, R139, R140, R141, R142, R151, R157, R158, R59: device teg2:0603 -> passive:0603
- C153, C154: value 100n -> 100nF; device teg2:0603 -> passive:0402
- C155, C156, C160, R152, R7, R90: device teg2:0603 -> passive:0402
- C157, C158, C159, C161: value 100µF -> 100uF
- C163, C174, C85, C95: value 22pF -> 15pF
- C164: value 100uF -> 470nF
- C166: value 470nF -> 100uF
- C168, C169, C170, C175, C176, C2, C3, C79, C80, C82, C88, C92, C93: value 10µF -> 10uF
- C172, C190, C195, C36, C37, C39, C40, C41, C42, C45, C47, C49, C50, C52, C53, C54, C83, C87, C91: device passive:0603 -> passive:0402
- C51: device rcl:C0603K -> passive:0402
- IC1, IC10: value TPS62560 -> TPS62240DDC
- IC11, IC12, IC29, IC7: value (none) -> TPS73001DBVR
- IC22: value 4052D -> 74HC4052D
- IC25: value ADS1112 -> INA331IDGK; device teg4:MSOP10 -> amplifiers-and-linear:MSOP08
- L10, L11, L8, L9: value (none) -> 220nH
- L4, L5: device rcl:L3216C -> passive:0603
- R1, R2: value 100 -> 100R; device teg2:0603 -> passive:0402
- R100, R101, R102, R103, R79, R97, R98, R99: value 47 -> 47R
- R105, R56, R57, R94: value 200 -> 200R
- R107, R46, R47: value 360 -> 360k
- R108, R109, R110, R111: value 6k8 -> 4k7; device teg2:0603 -> passive:0402
- R112: value 360 -> 240k
- R116, R117, R118, R119, R120, R121, R122, R123: value 100 -> 100R
- R146, R150: value 220k -> 1M
- R153: value (none) -> 1M
- R154: value 1M -> 100k
- R155: value 100k -> 1k
- R156: value 1k -> 68R
- R159, R160: value 1.54k -> 1k5; device teg2:0603 -> passive:0603
- R161, R162: value 150 -> 150R; device teg2:0603 -> passive:0603
- R163, R166: value (none) -> 43k
- R164, R167: value (none) -> 30k
- R170: value 820k -> 75k
- R171: value 820k -> 22k
- R175: value (none) -> 75k
- R176: value (none) -> 24k
- R18: value 2k -> 2k2; device passive:0603 -> passive:0402
- R195: value 1k3 -> 910R
- R22, R23, R24, R25, R26, R27, R28, R29, R30, R31, R32, R33, R34, R35, R36, R37: value 51R -> 47R
- R3: value 1k -> 240R; device rcl:R0603 -> passive:0603
- R38, R39, R40, R41, R42, R43, R44, R45: value 47 -> 47R; device passive:0603 -> passive:0402
- R5: value 22R -> 47R
- R52: value 820k -> 43k
- R53: value 820k -> 39k
- R54: value (none) -> 36k
- R55: value (none) -> 27k
- R6: value 24k -> 4k7
- R60: value 4k7 -> NC; device teg2:0603 -> passive:0402
- R86: value 600R -> 100R; device teg2:0603 -> passive:0402
- R87: value 600R -> 68R; device teg2:0603 -> passive:0603
- SV1: value (none) -> 2x5 Pinheader
- SV2, SV3, SV4: value (none) -> 2x8 Pinheader
- moved L8 453.6 mm to (101.5, 61.9), turned to 270 degrees
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Connections:
- removed net -2V5: C176.1, C198.2, R174.2
- removed net GPSPICLK: U2.M12
- removed net GPSPICS: U2.N12
- removed net GPSPIDATA: U2.M11
- removed net LAD13OO: U2.P11
- removed net N$148: IC25.5, R111.2
- removed net SCL: IC25.8, R59.2
- removed net SDA: IC25.7, R60.2, U2.P8
- removed net V-: IC31.4
- new net -2V5A: C176.1, C198.2, C207.1, C209.1, C219.1, C232.1, C234.1, C244.1, IC31.4, IC34.7, IC35.7, IC36.4, IC39.7, IC40.7, IC41.4, R174.2
- new net ATTRL+: IC37.1, R234.2
- new net ATTRL+B: IC42.1, R270.2
- new net ATTRL-: IC37.15, R236.1
- new net ATTRL-B: IC42.15, R272.1
- new net AUXIN: IC34.11, R275.2
- new net AUXINCH0: IC25.6, IC39.11, R202.2
- new net AUXOUT: R239.2
- new net CMP_MEAS_SEL: IC20.4, U2.R16
- new net DCRL+: IC37.3, R235.2
- new net DCRL+B: IC42.3, R271.2
- new net DCRL-: IC37.2, R233.1
- new net DCRL-B: IC42.2, R269.1
- new net DC_CS: IC32.2, U2.M14
- new net DC_DOUT: R280.1, R281.1, U2.T12
- new net GMUXA: IC34.10, IC37.4
- new net GMUXAB: IC39.10, IC42.4
- new net GMUXB: IC34.9, IC37.5
- new net GMUXBB: IC39.9, IC42.5
- new net GMUXC: IC35.10, IC37.6
- new net GMUXCB: IC40.10, IC42.6
- new net GMUXD: IC35.9, IC37.7
- new net GMUXDB: IC40.9, IC42.7
- new net HFDAC: R282.2, SV4.11
- new net HFDAC_CLK: IC44.11, U2.F13
- new net HFDAC_CS: IC44.12, U2.J13
- new net HFDAC_DI: IC44.14, U2.L13
- new net N$222: IC20.16, R201.1
- new net N$224: IC20.6, R60.1
- new net N$225: IC25.1, R202.1, R203.2
- new net N$226: IC25.3, R204.2, R207.2
- new net N$227: IC25.2, R205.2, R206.1
- new net N$228: R204.1, SV5.3
- new net N$229: R205.1, SV5.1
- new net N$230: IC33.6, R208.1, R209.2
- new net N$231: IC33.7, R208.2, R211.2
- new net N$232: R209.1, R210.2
- new net N$233: IC33.9, R212.1, R213.2
- new net N$234: IC33.13, R215.1, R216.2
- new net N$235: IC33.14, R215.2, R217.2
- new net N$236: IC33.5, IC34.12, IC35.15, IC35.5, R220.2, R231.1
- new net N$237: IC33.8, R212.2, R214.2
- new net N$238: IC35.1, IC35.11, R211.1
- new net N$239: IC33.12, IC35.13, R219.2
- new net N$240: IC34.14, IC35.12, R214.1
- new net N$241: IC34.15, R217.1
- new net N$242: IC33.10, IC35.3, R218.2
- new net N$243: C211.2, K1.3, R241.1
- new net N$244: C211.1, K1.2, K2.3
- new net N$245: R221.2, R223.1
- new net N$246: C212.2, C214.1, C228.1, R221.1, R222.2, R242.2
- new net N$247: R222.1, R224.2
- new net N$248: C214.2, C223.2, C228.2, K2.4, R223.2
- new net N$249: R225.2, R227.1
- new net N$250: R226.1, R228.2
- new net N$251: C217.2, C222.2, C229.2, K2.2, R227.2
- new net N$252: IC36.2, R229.1, R230.2
- new net N$253: IC36.1, R229.2, R231.2
- new net N$254: IC34.13, IC36.5
- new net N$255: C224.1, R232.1, T2.3, T3.3, T4.3, T8.3
- new net N$256: K1.8, T3.2, T6.E
- new net N$257: K1.1, T2.2, T5.E
- new net N$258: R235.1, T2.1, T5.B
- new net N$259: R233.2, T3.1, T6.B
- new net N$260: K2.1, T4.2, T7.E
- new net N$261: K2.8, T8.2, T9.E
- new net N$262: R234.1, T4.1, T7.B
- new net N$263: R236.2, T8.1, T9.B
- new net N$264: IC36.7, R237.2, R238.2, R239.1
- new net N$265: IC36.3, K2.6
- new net N$266: C216.1, C222.1
- new net N$267: C213.1, C223.1
- new net N$268: IC36.6, R238.1
- new net N$269: C220.2, L12.1, R230.1
- new net N$270: C215.2, C217.1, C229.1, R225.1, R226.2, R243.2
- new net N$271: R240.2, X2.2
- new net N$272: R241.2, X2.1
- new net N$273: K2.5, R242.1
- new net N$274: K2.7, R243.1
- new net N$281: IC38.6, R244.1, R245.2
- new net N$282: IC38.7, R244.2, R247.2
- new net N$283: R245.1, R246.2
- new net N$284: IC38.9, R248.1, R249.2
- new net N$285: IC38.13, R251.1, R252.2
- new net N$286: IC38.14, R251.2, R253.2
- new net N$287: IC38.5, IC39.12, IC40.15, IC40.5, R256.2, R267.1
- new net N$288: IC38.8, R248.2, R250.2
- new net N$289: IC40.1, IC40.11, R247.1
- new net N$290: IC38.12, IC40.13, R255.2
- new net N$291: IC39.14, IC40.12, R250.1
- new net N$292: IC39.15, R253.1
- new net N$293: IC38.10, IC40.3, R254.2
- new net N$294: C236.2, K3.3, R277.1
- new net N$295: C236.1, K3.2, K4.3
- new net N$296: R257.2, R259.1
- new net N$297: C237.2, C239.1, C253.1, R257.1, R258.2, R278.2
- new net N$298: R258.1, R260.2
- new net N$299: C239.2, C248.2, C253.2, K4.4, R259.2
- new net N$300: R261.2, R263.1
- new net N$301: R262.1, R264.2
- new net N$302: C242.2, C247.2, C254.2, K4.2, R263.2
- new net N$303: IC41.2, R265.1, R266.2
- new net N$304: IC41.1, R265.2, R267.2
- new net N$305: IC39.13, IC41.5
- new net N$306: C249.1, R268.1, T10.3, T11.3, T14.3, T16.3
- new net N$307: K3.8, T11.2, T13.E
- new net N$308: K3.1, T10.2, T12.E
- new net N$309: R271.1, T10.1, T12.B
- new net N$310: R269.2, T11.1, T13.B
- new net N$311: K4.1, T14.2, T15.E
- new net N$312: K4.8, T16.2, T17.E
- new net N$313: R270.1, T14.1, T15.B
- new net N$314: R272.2, T16.1, T17.B
- new net N$315: IC41.7, R273.2, R274.2, R275.1
- new net N$316: IC41.3, K4.6
- new net N$317: C241.1, C247.1
- new net N$318: C238.1, C248.1
- new net N$319: IC41.6, R274.1
- new net N$320: C245.2, L14.1, R266.1
- new net N$321: C240.2, C242.1, C254.1, R261.1, R262.2, R279.2
- new net N$322: R276.2, X3.2
- new net N$323: R277.2, X3.1
- new net N$324: K4.5, R278.1
- new net N$325: K4.7, R279.1
- new net N$332: IC32.9, R280.2
- new net N$333: R284.1, R285.1, R286.2
- new net N$334: R286.1, R287.2, R293.1
- new net N$335: R287.1, R288.2, R294.1
- new net N$336: R288.1, R289.2, R295.1
- new net N$337: R289.1, R290.2, R296.1
- new net N$338: R290.1, R291.2, R297.1
- new net N$339: R291.1, R292.2, R298.1
- new net N$340: R292.1, R299.2
- new net N$341: IC43.1, R283.2, R284.2
- new net N$342: IC44.15, R283.1
- new net N$343: IC44.1, R285.2
- new net N$344: IC44.2, R293.2
- new net N$345: IC44.3, R294.2
- new net N$346: IC44.4, R295.2
- new net N$347: IC44.5, R296.2
- new net N$348: IC44.6, R297.2
- new net N$349: IC44.7, R298.2
- new net N$350: IC43.3, R300.1
- new net N$351: IC43.4, R282.1, R300.2
- new net PULLUP1XA: R89.2, U2.T11
- new net SPICHAIN: IC37.9, IC42.14
- new net SPICHAINB: IC42.9
- new net SPICLK: IC37.11, IC42.11, U2.A13
- new net SPICS: IC37.12, IC42.12, U2.B14
- new net SPIDI: IC37.14, U2.A14
- net +3.6V: no longer IC31.8
- net +3V3: no longer R59.1, R60.1
- net +5V: now also C139.1, C204.2, C205.2, C206.2, C208.2, C210.2, C221.2, C230.2, C231.2, C233.2, C235.2, C246.2, C255.1, C256.1, IC25.7, IC25.8, IC32.8, IC33.4, IC34.16, IC35.16, IC37.10, IC37.16, IC38.4, IC39.16, IC40.16, IC42.10, IC42.16, IC43.5, IC44.10, IC44.16, R232.2, R268.2
- net 3V3A: now also C218.2, C243.2, IC31.8, IC36.8, IC41.8; no longer C139.1, IC25.6
- net AINL: now also SV4.8; no longer SV4.10
- net AINR: now also SV4.7; no longer SV4.9
- net AUBIAS: now also IC15.3; no longer IC15.2
- net AUPDN: now also U2.R15
- net AU_CCLK: now also IC32.1, U2.T14
- net AU_CDTI: now also IC32.10, U2.T15
- net AU_CSN: now also U2.T13
- net AU_OVFL: now also U2.R14
- net AU_OVFR: now also U2.M15
- net AVREFM: now also C225.1, C226.1, C227.1, C250.1, C251.1, C252.1, IC25.5, R203.1, R206.2, R207.1, R210.1, R213.1, R216.1, R218.1, R219.1, R220.1, R246.1, R249.1, R252.1, R254.1, R255.1, R256.1
- net CMPMEAS_+: now also R59.2; no longer IC20.11
- net CMPMEAS_A: now also U2.R12
- net CMPMEAS_B: now also U2.M13
- net CMPMEAS_EN: now also U2.N12
- net EXVO: now also R111.1
- net EXVOI: now also C189.2
- net GND: now also C148.2, C150.1, C201.2, C202.2, C203.2, C204.1, C205.1, C206.1, C207.2, C208.1, C209.2, C210.1, C212.1, C213.2, C215.1, C216.2, C218.1, C219.2, C220.1, C221.1, C224.2, C225.2, C226.2, C227.2, C230.1, C231.1, C232.2, C233.1, C234.2, C235.1, C237.1, C238.2, C240.1, C241.2, C243.1, C244.2, C245.1, C246.1, C249.2, C250.2, C251.2, C252.2, C255.2, C256.2, IC20.1, IC22.8, IC25.4, IC31.2, IC31.3, IC32.3, IC33.1, IC33.11, IC33.2, IC33.3, IC34.6, IC34.8, IC35.6, IC35.8, IC37.13, IC37.8, IC38.1, IC38.11, IC38.2, IC38.3, IC39.6, IC39.8, IC40.6, IC40.8, IC42.13, IC42.8, IC43.2, IC44.13, IC44.8, R201.2, R224.1, R228.1, R240.1, R260.1, R264.1, R276.1, R281.2, R299.1, R3.2, R60.2, SV4.10, SV4.13, SV4.9, SV5.2, T12.C, T13.C, T15.C, T17.C, T5.C, T6.C, T7.C, T9.C; no longer IC25.10, IC25.3, IC25.9, R3.1, SV4.11, SV4.7, SV4.8
- net I2SBCK: now also U2.N16
- net I2SDATAIN: now also U2.M16; no longer U2.L8
- net I2SDATAOUT: now also U2.N14; no longer U2.L7
- net I2SLRCK: now also U2.P15
- net I2SSCLK: now also U2.P16; no longer R89.2, U2.T11
- net N$117: now also C203.1, IC32.4; no longer IC25.1
- net N$142: now also C202.1, IC32.5; no longer IC25.2
- net N$144: now also C201.1, IC32.6; no longer IC25.4
- net N$149: now also R3.1; no longer R3.2
- net N$152: now also IC15.2; no longer IC15.3
- net N$162: now also SV4.15; no longer SV4.13
- net N$163: now also SV4.16; no longer SV4.14
- net N$164: now also IC32.7, R111.2; no longer R110.1, SV4.15
- net N$165: now also R110.1, SV4.14; no longer R111.1, SV4.16
- net N$183: now also IC20.11, R59.1; no longer C148.2, C150.1, IC22.8
- net OFFSETCH0: now also L14.2
- net OFFSETCH1: now also L12.2
- net OUTPUTCH0: now also R273.1
- net OUTPUTCH1: now also R237.1
- net PWMEXVO: now also U2.D11
- net PWMLA: now also U2.E12
- net PWMLAVIO: now also U2.D12
- net PWMOFFS0: now also U2.C10
- net PWMOFFS1: now also U2.C11
Routing:
- net +5V: track 53.7 -> 380.4 mm, vias 4 -> 28
- net GND: track 275.4 -> 519.2 mm, vias 132 -> 236
- net EXVO: track 0.00 -> 228.7 mm, vias 0 -> 4
- net -2V5A: track 0.00 -> 212.5 mm, vias 0 -> 13
- net 3V3A: track 73.7 -> 270.4 mm, vias 11 -> 12
- net AVREFM: track 0.00 -> 189.0 mm, vias 0 -> 12
- net LAVIO: track 1.55 -> 186.8 mm, vias 0 -> 7
- net LOGICOFFSET: track 23.9 -> 190.5 mm, vias 8 -> 11
- net -5V: track 1.28 -> 155.3 mm, vias 0 -> 5
- net HFDAC: track 0.00 -> 98.8 mm, vias 0 -> 3
- net SPICS: track 0.00 -> 97.2 mm, vias 0 -> 3
- net SPICLK: track 0.00 -> 96.0 mm, vias 0 -> 3
- net 1V2REF: track 15.1 -> 106.7 mm, vias 3 -> 5
- net PWMLAVIO: track 0.00 -> 86.8 mm, vias 0 -> 2
- net HFDAC_CS: track 0.00 -> 78.8 mm, vias 0 -> 4
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- added copper zone on layer 3, net +5V
- added copper zone on layer 3, net GND
- added copper zone on layer 3, net N$275
- added copper zone on layer 3, net N$276
- added copper zone on layer 3, net N$277
- added copper zone on layer 1, net N$278
- added copper zone on layer 3, net N$279
- added copper zone on layer 3, net N$280
- added copper zone on layer 3, net N$326
- added copper zone on layer 3, net N$327
- added copper zone on layer 3, net N$328
- added copper zone on layer 1, net N$329
- added copper zone on layer 3, net N$330
- added copper zone on layer 3, net N$331
- added copper zone on layer 2, net N$352
- added copper zone on layer 2, net N$353
- added copper zone on layer 2, net N$354
Other:
- board size 128 x 411.1 mm -> 100 x 100.1 mm
- board text added: "LBF 0.5"
- board text removed: "SPSCOPE V1"

Commit message: Final oreder prototype
Routing:
- net VREFDDR: track 101.4 -> 100.4 mm
- added copper zone on layer 16, net VREFDDR
Other:
- board size 100 x 100.1 mm -> 100 x 99.8 mm
Changed lines of the file:
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@@
 <plain>
 <wire x1="60.2234" y1="0" x2="160.2032" y2="0" width="0" layer="20"/>
-<wire x1="160.2032" y1="0" x2="160.2032" y2="100.0508" width="0" layer="20"/>
-<wire x1="160.2032" y1="100.0508" x2="60.2234" y2="100.0762" width="0" layer="20"/>
-<wire x1="60.2234" y1="100.0762" x2="60.2234" y2="0" width="0" layer="20"/>
+<wire x1="160.2032" y1="0" x2="160.2282" y2="99.7508" width="0" layer="20"/>
+<wire x1="160.2282" y1="99.7508" x2="60.2484" y2="99.7762" width="0" layer="20"/>
+<wire x1="60.2484" y1="99.7762" x2="60.2234" y2="0" width="0" layer="20"/>
 <wire x1="119.0244" y1="58.0644" x2="119.0244" y2="57.8866" width="0" layer="47"/>
 <wire x1="83.6168" y1="22.1488" x2="83.4136" y2="22.1488" width="0" layer="47"/>
@@
 <vertex x="128.525" y="43.2"/>
 <vertex x="127.875" y="43.85"/>
-<vertex x="127.875" y="45.9875"/>
-<vertex x="128.2625" y="46.375"/>
-<vertex x="128.875" y="46.375"/>
-<vertex x="129.5125" y="47.0125"/>
-<vertex x="129.5125" y="49.8125"/>
-<vertex x="128.9375" y="49.975"/>
+<vertex x="127.9" y="45.7875"/>
+<vertex x="128.2375" y="46.175"/>
+<vertex x="129.175" y="46.175"/>
+<vertex x="129.175" y="46.525"/>
+<vertex x="129.0375" y="46.6625"/>
+<vertex x="128.5875" y="46.975"/>
+<vertex x="128.5375" y="49.775"/>
+<vertex x="128.375" y="49.9375"/>
 <vertex x="127.925" y="50"/>
 <vertex x="127.4875" y="50.3625"/>
@@
 <vertex x="129.725" y="55.0125"/>
 <vertex x="130.0125" y="54.575"/>
+<vertex x="129.95" y="51.2375"/>
+<vertex x="129.0125" y="50.225"/>
+<vertex x="129.0125" y="47.3125"/>
+<vertex x="129.975" y="46.35"/>
 <vertex x="129.975" y="45.7375"/>
 <vertex x="130.3625" y="45.35"/>
@@
 <via x="152.6865" y="18.7085" extent="1-16" drill="0.3048"/>
 <via x="151.003" y="23.9522" extent="1-16" drill="0.3048"/>
-<polygon width="0.254" layer="2" isolate="0.254">
+<polygon width="0.254" layer="2" isolate="0.15">
 <vertex x="137.2362" y="29.8704"/>
 <vertex x="136.9544" y="29.2612"/>
@@
 <via x="141.4526" y="18.288" extent="1-16" drill="0.3048"/>
 <via x="133.7726" y="19.3301" extent="1-16" drill="0.3048"/>
-<polygon width="0.2032" layer="3" isolate="0.254">
+<polygon width="0.2032" layer="3" isolate="0.15">
 <vertex x="152.2984" y="29.845"/>
 <vertex x="148.6662" y="29.8704"/>
@@
 <wire x1="156.45" y1="56.9999" x2="156.727" y2="57.0125" width="0.6096" layer="1"/>
 <contactref element="R50" pad="2"/>
-<polygon width="0.4064" layer="3" isolate="0.254">
-<vertex x="132.9625" y="42.6"/>
+<polygon width="0.4064" layer="3" isolate="0.15">
+<vertex x="132.4875" y="44.2625"/>
+<vertex x="131.8375" y="44.3"/>
+<vertex x="131.575" y="44.5625"/>
+<vertex x="129.425" y="44.5625"/>
+<vertex x="132.9375" y="41.05"/>
 <vertex x="132.9375" y="41"/>
 <vertex x="134.15" y="39.6125"/>
@@
 <vertex x="132.8375" y="49.8875"/>
 <vertex x="133.025" y="46.9375"/>
-<vertex x="132.95" y="43.625"/>
+<vertex x="133.05" y="44.675"/>
 </polygon>
 <wire x1="143.475" y1="35.4499" x2="143.475" y2="37.2125" width="0.6096" layer="1"/>
@@
 <wire x1="155.6625" y1="50.9375" x2="158.125" y2="50.9375" width="0.15" layer="1"/>
 <wire x1="158.125" y1="50.9375" x2="158.675" y2="51.4875" width="0.15" layer="1"/>
-<wire x1="148.65" y1="53.375" x2="148.3875" y2="53.375" width="0.15" layer="1"/>
-<wire x1="148.3875" y1="53.375" x2="148.3" y2="53.2875" width="0.15" layer="1"/>
-<wire x1="148.3" y1="53.2875" x2="145.7875" y2="53.2875" width="0.15" layer="1"/>
+<wire x1="148.65" y1="53.375" x2="148.5125" y2="53.375" width="0.15" layer="1"/>
+<wire x1="148.5125" y1="53.375" x2="148.425" y2="53.2875" width="0.15" layer="1"/>
+<wire x1="148.425" y1="53.2875" x2="145.7875" y2="53.2875" width="0.15" layer="1"/>
 <wire x1="145.7875" y1="53.2875" x2="145.425" y2="52.9375" width="0.15" layer="1"/>
 <wire x1="145.425" y1="52.9375" x2="145.2875" y2="52.9375" width="0.15" layer="1"/>
-<wire x1="145.2875" y1="52.9375" x2="144.725" y2="52.175" width="0.15" layer="1"/>
-<via x="144.725" y="52.175" extent="1-16" drill="0.3"/>
-<wire x1="144.725" y1="52.175" x2="144.725" y2="53.125" width="0.15" layer="16"/>
-<wire x1="144.725" y1="53.125" x2="143.775" y2="54.225" width="0.3048" layer="16"/>
+<wire x1="145.2875" y1="52.9375" x2="145.4375" y2="52.9" width="0.15" layer="1"/>
+<via x="145.4375" y="52.9" extent="1-16" drill="0.3"/>
+<wire x1="145.4375" y1="52.9" x2="144.725" y2="53.125" width="0.15" layer="16"/>
+<wire x1="144.725" y1="53.125" x2="144.725" y2="53.175" width="0.3048" layer="16"/>
+<wire x1="144.725" y1="53.175" x2="143.8375" y2="54.0625" width="0.3048" layer="16"/>
+<wire x1="143.8375" y1="54.0625" x2="143.775" y2="54.225" width="0.3048" layer="16"/>
 <via x="143.775" y="54.225" extent="1-16" drill="0.3"/>
 <wire x1="143.775" y1="54.225" x2="143.775" y2="56.925" width="0.3048" layer="1"/>
@@
 <vertex x="131.675" y="45.0125"/>
 </polygon>
-<wire x1="144.7605" y1="52.875" x2="144.7605" y2="52.2105" width="0.4064" layer="16"/>
-<wire x1="144.7605" y1="52.2105" x2="144.725" y2="52.175" width="0.4064" layer="16"/>
+<wire x1="144.7605" y1="52.875" x2="144.923" y2="52.898" width="0.4064" layer="16"/>
+<wire x1="144.923" y1="52.898" x2="145.4375" y2="52.9" width="0.4064" layer="16"/>
 <contactref element="R2" pad="2"/>
 <contactref element="R1" pad="1"/>
+<polygon width="0.15" layer="1" isolate="0.15">
+<vertex x="145.3125" y="52.7"/>
+<vertex x="145.6125" y="52.7"/>
+<vertex x="145.9" y="52.4125"/>
+<vertex x="146.3625" y="52.4125"/>
+<vertex x="146.9875" y="53.0375"/>
+<vertex x="148.5875" y="53.0375"/>
+<vertex x="148.9125" y="53.3625"/>
+<vertex x="148.9125" y="53.4625"/>
+<vertex x="148.6875" y="53.6875"/>
+<vertex x="148.225" y="53.6875"/>
+<vertex x="148.075" y="53.5375"/>
+<vertex x="145.425" y="53.5375"/>
+<vertex x="145.125" y="53.2375"/>
+<vertex x="145.125" y="52.8875"/>
+</polygon>
+<polygon width="0.15" layer="1" isolate="0.15">
+<vertex x="143.7875" y="54.2"/>
+<vertex x="144.175" y="54.2"/>
+<vertex x="144.375" y="54.4"/>
+<vertex x="144.375" y="57.5125"/>
+<vertex x="143.9125" y="57.975"/>
+<vertex x="143.55" y="57.975"/>
+<vertex x="143.3625" y="57.7875"/>
+<vertex x="143.3625" y="54.575"/>
+<vertex x="143.7375" y="54.2"/>
+</polygon>
+<polygon width="0.15" layer="16" isolate="0.15">
+<vertex x="136.725" y="57.25"/>
+<vertex x="143.6625" y="57.25"/>
+<vertex x="144.075" y="57.6625"/>
+<vertex x="144.075" y="58.05"/>
+<vertex x="143.95" y="58.175"/>
+<vertex x="136.775" y="58.175"/>
+<vertex x="136.5125" y="57.9125"/>
+<vertex x="136.5125" y="57.5"/>
+<vertex x="136.75" y="57.2625"/>
+</polygon>
 </signal>
 <signal name="CASN">
@@
 <wire x1="132.15" y1="52.3375" x2="132.6625" y2="51.9" width="0.15" layer="16"/>
 <wire x1="150.25" y1="51.775" x2="150.25" y2="51.7875" width="0.15" layer="1"/>
-<via x="145.525" y="52.1625" extent="1-16" drill="0.3"/>
-<wire x1="145.525" y1="52.1625" x2="145.4625" y2="52.1" width="0.15" layer="16"/>
-<wire x1="145.525" y1="52.1625" x2="145.525" y2="52.3" width="0.15" layer="1"/>
-<wire x1="145.525" y1="52.3" x2="146.2" y2="52.975" width="0.15" layer="1"/>
-<wire x1="146.2" y1="52.975" x2="148.8875" y2="52.975" width="0.15" layer="1"/>
+<via x="145.5" y="52.1375" extent="1-16" drill="0.3"/>
+<wire x1="145.5" y1="52.1375" x2="145.4625" y2="52.1" width="0.15" layer="16"/>
 <wire x1="148.8875" y1="52.975" x2="149.05" y2="52.8125" width="0.15" layer="1"/>
 <wire x1="149.05" y1="52.8125" x2="149.05" y2="52.4" width="0.15" layer="1"/>
@@
 <wire x1="135.9125" y1="50.4375" x2="136.15" y2="50.2" width="0.15" layer="16"/>
 <wire x1="136.15" y1="50.2" x2="143.5625" y2="50.2" width="0.15" layer="16"/>
-<wire x1="143.5625" y1="50.2" x2="145.525" y2="52.1625" width="0.15" layer="16"/>
+<wire x1="143.5625" y1="50.2" x2="145.5" y2="52.1375" width="0.15" layer="16"/>
+<wire x1="145.5" y1="52.1375" x2="146.3875" y2="52.1375" width="0.15" layer="1"/>
+<wire x1="146.3875" y1="52.1375" x2="147.05" y2="52.8" width="0.15" layer="1"/>
+<wire x1="147.05" y1="52.8" x2="147.6875" y2="52.8" width="0.15" layer="1"/>
+<wire x1="147.6875" y1="52.8" x2="147.75" y2="52.8625" width="0.15" layer="1"/>
+<wire x1="147.75" y1="52.8625" x2="148.1875" y2="52.8625" width="0.15" layer="1"/>
+<wire x1="148.1875" y1="52.8625" x2="148.3" y2="52.975" width="0.15" layer="1"/>
+<wire x1="148.3" y1="52.975" x2="148.8875" y2="52.975" width="0.15" layer="1"/>
 </signal>
 <signal name="RASN">
