File: schpcb/LabFriendMain1.brd (EAGLE design)
At the start: 100 x 99.8 mm, 654 parts, among them IC1 TPS62240DDC, IC10 TPS62240DDC, IC11 TPS73001DBVR, IC12 TPS73001DBVR, IC13 AK4621, IC14 TPS72301, IC15 LME49721, IC16 NE5532, IC17 OPA2134, IC18 LM8272, IC19 LMV358MM, IC2 25px80, IC20 ISL54405IRTZ, IC21 NE5532, IC22 74HC4052D, IC23 LME49721, IC24 74HC00D, IC25 INA331IDGK, IC26 MT41J128M8, IC27 74HCT132D, IC28 TPS72301, IC29 TPS73001DBVR, IC3 SI8462, IC30 LM8272, IC31 LMV358MM, IC32 ADS1118IDGSR, IC33 ADA4853-3RU, IC34 4052D, IC35 4052D, IC36 OPA2354, IC37 74HC595D, IC38 ADA4853-3RU, IC39 4052D, IC4 FT232H, IC40 4052D, IC41 OPA2354, IC42 74HC595D, IC43 LM321MF, IC44 74HC595D, IC5 ADC08200, IC6 ADC08200, IC7 TPS73001DBVR, IC8 93LC56SM, IC9 74LVC8T245, K1 G6K-2F-Y, K2 G6K-2F-Y, K3 G6K-2F-Y, K4 G6K-2F-Y, Q1 12MHz, Q2 FDN335N, Q3 FDN335N, T1 EFD15DCDCPM5P33EFD15, T10 BC850, T11 BC850, T12 BC856ASMD, T13 BC856ASMD, T14 BC850, T15 BC856ASMD, T16 BC850, T17 BC856ASMD, T2 BC850, T3 BC850, T4 BC850, T5 BC856ASMD, T6 BC856ASMD, T7 BC856ASMD, T8 BC850, T9 BC856ASMD, U2 6SLX9FTG256, X1 MINI-USB-32005-201, X2 31-5431-10RFX, X3 31-5431-10RFX

Commit message: many improovments and bugfixes and added features
Parts:
- R261: value 51k -> 130k
- R262: value 39k -> 47k
- R263: value 910k -> 820k
- R264: value 1k -> 3k
Changed lines of the file:
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@@
 <?xml version="1.0" encoding="utf-8"?>
 <!DOCTYPE eagle SYSTEM "eagle.dtd">
-<eagle version="7.3.0">
+<eagle version="7.7.0">
 <drawing>
 <settings>
@@
 <attribute name="NAME" x="63.3316" y="75.4962" size="0.6096" layer="25" ratio="10"/>
 </element>
-<element name="R261" library="passive" package="0603" value="51k" x="74.7616" y="63.5328" smashed="yes" rot="R90">
+<element name="R261" library="passive" package="0603" value="130k" x="74.7616" y="63.5328" smashed="yes" rot="R90">
 <attribute name="VALUE" x="72.8566" y="62.3898" size="0.8128" layer="27" ratio="10" rot="R90"/>
 <attribute name="NAME" x="75.0918" y="62.4914" size="0.6096" layer="25" ratio="10" rot="R90"/>
@@
 <attribute name="NAME" x="75.676" y="64.5996" size="0.6096" layer="25" ratio="10" rot="R270"/>
 </element>
-<element name="R262" library="passive" package="0603" value="39k" x="75.041" y="61.5516" smashed="yes">
+<element name="R262" library="passive" package="0603" value="47k" x="75.041" y="61.5516" smashed="yes">
 <attribute name="VALUE" x="73.898" y="63.4566" size="0.8128" layer="27" ratio="10"/>
 <attribute name="NAME" x="73.9742" y="61.2468" size="0.6096" layer="25" ratio="10"/>
@@
 <attribute name="VALUE" x="60.3344" y="66.3776" size="1.27" layer="27" rot="R270"/>
 </element>
-<element name="R263" library="passive" package="0603" value="910k" x="73.977790625" y="65.49746875" smashed="yes" rot="R180">
+<element name="R263" library="passive" package="0603" value="820k" x="73.977790625" y="65.49746875" smashed="yes" rot="R180">
 <attribute name="VALUE" x="75.12079375" y="63.59246875" size="0.8128" layer="27" ratio="10" rot="R180"/>
 <attribute name="NAME" x="72.89865625" y="65.204996875" size="0.6096" layer="25" ratio="10"/>
 </element>
-<element name="R264" library="passive" package="0603" value="1k" x="72.247" y="61.5516" smashed="yes">
+<element name="R264" library="passive" package="0603" value="3k" x="72.247" y="61.5516" smashed="yes">
 <attribute name="VALUE" x="71.104" y="63.4566" size="0.8128" layer="27" ratio="10"/>
 <attribute name="NAME" x="71.7898" y="61.2722" size="0.6096" layer="25" ratio="10"/>
@@
 <contactref element="SV1" pad="3"/>
 <contactref element="R9" pad="2"/>
-<contactref element="IC2" pad="4"/>
 <contactref element="C33" pad="2"/>
 <contactref element="C34" pad="2"/>
@@
 <contactref element="C185" pad="2"/>
 <contactref element="C187" pad="2"/>
-<contactref element="C187" pad="2"/>
-<contactref element="C186" pad="2"/>
 <contactref element="C186" pad="2"/>
 <contactref element="IC30" pad="4"/>
@@
 <wire x1="94.6967" y1="76.2582" x2="95.1539" y2="75.9534" width="0.4064" layer="16"/>
 <wire x1="93.7823" y1="66.3776" x2="94.1125" y2="66.403" width="0.4064" layer="16"/>
-<contactref element="IC37" pad="8"/>
 <contactref element="C221" pad="1"/>
 <wire x1="83.1905" y1="38.3522" x2="81.9205" y2="38.3522" width="0.6096" layer="1"/>
@@
 <wire x1="76.5142" y1="76.2582" x2="76.9714" y2="75.9534" width="0.4064" layer="16"/>
 <wire x1="75.5998" y1="66.3776" x2="75.93" y2="66.403" width="0.4064" layer="16"/>
-<contactref element="IC42" pad="8"/>
 <contactref element="C246" pad="1"/>
 <wire x1="65.008" y1="38.3522" x2="63.738" y2="38.3522" width="0.6096" layer="1"/>
@@
 <contactref element="C51" pad="1"/>
 <contactref element="IC4" pad="46"/>
-<contactref element="IC4" pad="24"/>
-<contactref element="IC4" pad="12"/>
 <contactref element="R16" pad="2"/>
 <contactref element="R19" pad="2"/>
